File: mcu.kicad_sch (KiCad schematic)
At the start: 6 parts, among them J2 Conn_01x03_Male, J3 Conn_01x02_Male, J4 Conn_ARM_JTAG_SWD_10, U2 STM32L011F4Px

Commit message: Gerbers
Changed lines of the file:
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@@
-    (stroke (width 0) (type default) (color 0 0 0 0))
-  )
-  (wire (pts (xy 71.12 158.75) (xy 66.04 158.75))
     (stroke (width 0) (type default) (color 0 0 0 0))
   )
@@
     (stroke (width 0) (type default) (color 0 0 0 0))
   )
+  (wire (pts (xy 66.04 158.75) (xy 71.12 158.75))
+    (stroke (width 0) (type default) (color 0 0 0 0))
+  )
   (wire (pts (xy 53.34 143.51) (xy 53.34 142.24))
     (stroke (width 0) (type default) (color 0 0 0 0))
@@
   )
   (wire (pts (xy 55.88 71.12) (xy 53.34 71.12))
-    (stroke (width 0) (type default) (color 0 0 0 0))
-  )
-  (wire (pts (xy 71.12 156.21) (xy 66.04 156.21))
     (stroke (width 0) (type default) (color 0 0 0 0))
   )
@@
     (stroke (width 0) (type default) (color 0 0 0 0))
   )
-  (wire (pts (xy 71.12 151.13) (xy 66.04 151.13))
-    (stroke (width 0) (type default) (color 0 0 0 0))
-  )
   (wire (pts (xy 66.04 107.95) (xy 78.74 107.95))
     (stroke (width 0) (type default) (color 0 0 0 0))
   )
   (wire (pts (xy 76.2 82.55) (xy 78.74 82.55))
+    (stroke (width 0) (type default) (color 0 0 0 0))
+  )
+  (wire (pts (xy 66.04 156.21) (xy 71.12 156.21))
     (stroke (width 0) (type default) (color 0 0 0 0))
   )
@@
     (stroke (width 0) (type default) (color 0 0 0 0))
   )
+  (wire (pts (xy 66.04 151.13) (xy 71.12 151.13))
+    (stroke (width 0) (type default) (color 0 0 0 0))
+  )

Commit message: Add THT debug
Parts:
- J4: footprint Connector_PinHeader_1.27mm:PinHeader_2x05_P1.27mm_Vertical_SMD -> Connector_PinHeader_1.27mm:PinHeader_2x05_P1.27mm_Vertical
Changed lines of the file:
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@@
       (effects (font (size 1.27 1.27)) (justify right))
     )
-    (property "Footprint" "Connector_PinHeader_1.27mm:PinHeader_2x05_P1.27mm_Vertical_SMD" (id 2) (at 53.34 158.75 0)
+    (property "Footprint" "Connector_PinHeader_1.27mm:PinHeader_2x05_P1.27mm_Vertical" (id 2) (at 53.34 158.75 0)
       (effects (font (size 1.27 1.27)) hide)
     )
