File: neopixels.kicad_sch (KiCad schematic)
At the start: 20 parts

Commit message: Prod
Parts:
- removed D11, D12, D13, D14, D15, D16, D17, D18, D19, D20: WS2813B, Library:LED_WS2813_hand, symbol pumpkin syms:WS2813B
